File: gp-mpu.kicad_pcb (KiCad board)
At the start: 2 copper layers, 302.1 x 188.2 mm, 216 parts, among them J1 Power, J2 Lamp, J3 BDU DISPLAY, J4 Sound, J5 Switch Matrix, J6 Cabinet, J7 Solenoid, J9 DISPLAY, Q1 2N3904, SW1 SW_DIP_x04, SW2 Dip 1-8, SW3 Dip 9-16, SW4 Dip 17-24, SW5 Dip 25-32, SW6 Reset, U1 Z80-CTC, U10 74LS138, U11 74LS138, U12 74LS00, U13 74LS377, U14 74LS377, U15 MIC1232, U16 LM339, U17 74LS138, U18 7416, U19 LM339, U2 Z80CPU, U20 LM339, U3 74LS04, U4 74LS32, U5 74LS00, U6 27C020, U7 FM16W08-SG, U8 8255, U9 7417, Y1 2.4576mhz

Commit message: updates
Parts:
- added BT1: Battery_Cell, Battery:BatteryHolder_ComfortableElectronic_CH273-2450_1x2450, F.Cu at (198.0, 17.0)
- added D59: 1N5817*, Diode_THT:D_DO-41_SOD81_P10.16mm_Horizontal, F.Cu at (189.2, 24.6)
- added D60: 1N4148*, Diode_THT:D_DO-35_SOD27_P7.62mm_Horizontal, F.Cu at (193.5, 24.6)
- added J8: Ext Battery (when using 6264), Connector_PinHeader_2.54mm:PinHeader_1x03_P2.54mm_Vertical, F.Cu at (238.5, 11.2)
- U7: value FM16W08-SG -> FM16W08-SG or 6264*
Connections:
- U7 pad 26: (no net) -> +BATT
- U7 pad 28: +5V -> +BATT
Routing:
- net +BATT: track 0.00 -> 179.1 mm, vias 0 -> 2
- net Net-(BT1-Pad1): track 0.00 -> 47.8 mm, vias 0 -> 1
- net GND: track 2366.1 -> 2403.4 mm, vias 7 -> 11
- net +5V: track 1472.6 -> 1497.9 mm
- net DISP+: track 962.3 -> 976.6 mm, vias 5 -> 19
- net DISP_GND: track 413.5 -> 419.5 mm, vias 3 -> 11
- net DISP_5V: track 415.8 -> 419.5 mm, vias 4 -> 11
- net PERIPH0_3: track 186.9 -> 183.2 mm
- net PERIPH0_2: track 192.4 -> 189.2 mm
- net PERIPH0_4: track 176.8 -> 173.6 mm
- net PERIPH0_1: track 159.7 -> 158.0 mm
Other:
- board text added: "* For NVRAM, install a jumper at D59 * D59 and D60 are only required when using battery backup, 6264 RAM"
- board text added: "*When using a 6264, install the battery section. If using NVRAM, install a jumper at D59."
- board text added: "+|GND|+"
- board text added: "0=Off, 1=On 1234 ---- 0000 - Sharp Shooter, Sharp Shooter 2 Coney Island!, Lizard 0001 - Super Nova 0010 - Global Warfare 0011 - Attila the Hun 0100 - Agents 777 0110 - Captain Hook 0111 - Andromeda 1000 - Cyclopes 1001 - Cocktail 110: Foxy Lady, Real, Rio, Black Velvet, Camel Lights 1010 - Cocktail 120: Star Trip, Family Fun! 1100 - Cocktail 140: Vegas 1110 - Cocktail 830: Lady Sharpshooter 1111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"
- board text added: "GamePlan MPU ver 1.3 github.com/jfleitz/gp-mpu"
- board text removed: "0=Off, 1=On 1234 ---- 0000 - Sharp Shooter, Sharp Shooter 2 Coney Island!, Lizard 0001 - Super Nova 0010 - Global Warfare 0011 - Attila the Hun 0100 - Agents 777 0110 - Captain Hook 0111 - Andromeda 1000 - Cyclopes 1001 - Cocktail 110: Foxy Lady, Real, Rio, Black Velvet, Camel Lights, Chuck-A-Luck 1010 - Cocktail 120: Star Trip, Family Fun! 1100 - Cocktail 140: Vegas 1110 - Cocktail 830: Lady Sha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"
- board text removed: "GamePlan MPU github.com/jfleitz/gp-mpu"

Commit message: enlarge all vias
Routing:
- net DIP_STROBE3: track 92.0 -> 92.8 mm
- net ADDR4: track 299.5 -> 298.8 mm
- net PC0: track 173.9 -> 174.6 mm
- net DISP_CLK2: track 300.8 -> 301.4 mm
- net LAMP_EN4: track 227.6 -> 227.0 mm
- net DISP_CLK4: track 520.8 -> 521.3 mm
Other:
- outline, holes or cut-outs redrawn
- board text added: "GamePlan MPU ver 1.4 github.com/jfleitz/gp-mpu"
- board text removed: "GamePlan MPU ver 1.3 github.com/jfleitz/gp-mpu"

Commit message: Update BDU connector
Parts:
- added JP1: NVRAM, Jumper:SolderJumper-2_P1.3mm_Open_RoundedPad1.0x1.5mm, F.Cu at (188.6, 28.5)
- BT1: value Battery_Cell -> 2732 coin cell
- D59: value 1N5817* -> 1N5817
- D60: value 1N4148* -> 1N4148
- J8: value Ext Battery (when using 6264) -> Ext Battery
- TP2: value TestPoint -> RST
- TP3: value TestPoint -> /RST
- U7: value FM16W08-SG or 6264* -> FM16W08-SG
Connections:
- J3 pad 1: DISP_CLK4 -> DISP_CLK5
- J3 pad 2: DISP_CLK2 -> DISP_CLK3
- J3 pad 22: unconnected-(J3-Pad22) -> PERIPH_EN
- J3 pad 3: DISP_CLK3 -> DISP_CLK4
- J3 pad 4: DISP_CLK1 -> DISP_CLK2
Routing:
- net DISP_CLK1: track 390.0 -> 173.2 mm, vias 5 -> 1
- net DISP_CLK5: track 160.9 -> 351.0 mm, vias 2 -> 6
- net PERIPH_EN: track 299.7 -> 417.8 mm, vias 2 -> 4
- net +5V: track 1497.8 -> 1510.6 mm
- net +BATT: track 179.1 -> 183.0 mm
- net DISP_CLK4: track 521.3 -> 523.3 mm
- net DISP_CLK3: track 315.7 -> 317.0 mm, vias 7 -> 6
- net DISP_CLK2: track 301.4 -> 300.3 mm
Other:
- board text added: "* For NVRAM, install a jumper at JP1 * D59 and D60 are only required when using battery backup, 6264 RAM"
- board text added: "+12V"
- board text added: "+24V"
- board text added: "+5V"
- board text added: "1"
- board text added: "12"
- board text added: "2"
- board text added: "25"
- board text added: "26"
- board text added: "9"
- board text added: "A"
- board text added: "ADDR1"
- board text added: "ADDR2"
- board text added: "ADDR3"
- board text added: "ADDR4"
- board text added: "BDU DISPLAY"
- board text added: "Bit0"
- board text added: "Bit1"
- board text added: "Bit2"
- board text added: "Bit3"
- board text added: "Disp +"
- board text added: "Disp +5v"
- board text added: "Disp+"
- board text added: "Disp5V"
- board text added: "DispGnd"
- board text added: "Dist GND"
- board text added: "GND"
- board text added: "GamePlan MPU ver 1.5 github.com/jfleitz/gp-mpu"
- board text added: "Gnd"
- board text added: "Line0"
- board text added: "Line1"
- board text added: "Line2"
- board text added: "Line3"
- board text added: "Line4"
- board text added: "Line5"
- board text added: "Line6"
- board text added: "Line7"
- board text added: "LmpEn1"
- board text added: "LmpEn2"
- board text added: "LmpEn3"
- board text added: "LmpEn4"
- board text added: "N"
- board text added: "PC5"
- board text added: "PC6"
- board text added: "PC7"
- board text added: "Periph Enable"
- board text added: "Strobe0"
- board text added: "Strobe1"
- board text added: "Strobe2"
- board text added: "Strobe3"
- board text added: "Strobe4"
- board text added: "bit0"
- board text added: "bit1"
- board text added: "bit2"
- board text added: "bit3"
- board text added: "dig6"
- board text removed: "* For NVRAM, install a jumper at D59 * D59 and D60 are only required when using battery backup, 6264 RAM"
- board text removed: "GamePlan MPU ver 1.4 github.com/jfleitz/gp-mpu"
