File: gp-mpu.kicad_sch (KiCad schematic)
At the start: 16 parts, among them SW1 SW_DIP_x04, U1 Z80-CTC, U2 Z80CPU, U3 74LS04, U4 74LS32, U5 74LS00, U6 27C020, U7 FM16W08-SG, U8 8255

Commit message: updates
Connections:
- net +5V: no longer U7.28 (VDD)
- new net +BATT: U7.26 (CE2), U7.28 (VDD)
Changed lines of the file:
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@@
     (comment 1 "github.com/jfleitz/gp-mpu")
+  )
+  (junction (at 212.09 21.59) (diameter 0) (color 0 0 0 0)
   )
   (junction (at 74.93 149.86) (diameter 0) (color 0 0 0 0)
@@
     (stroke (width 0) (type default) (color 0 0 0 0))
   )
+  (wire (pts (xy 208.28 21.59) (xy 212.09 21.59))
+    (stroke (width 0) (type default) (color 0 0 0 0))
+  )
   (wire (pts (xy 24.13 165.1) (xy 40.64 165.1))
     (stroke (width 0) (type default) (color 0 0 0 0))
@@
     (stroke (width 0) (type default) (color 0 0 0 0))
   )
+  (wire (pts (xy 212.09 21.59) (xy 212.09 25.4))
+    (stroke (width 0) (type default) (color 0 0 0 0))
+  )
   (wire (pts (xy 138.43 34.29) (xy 140.97 34.29))
     (stroke (width 0) (type default) (color 0 0 0 0))
@@
     (stroke (width 0) (type default) (color 0 0 0 0))
   )
+  (wire (pts (xy 208.28 24.13) (xy 208.28 21.59))
+    (stroke (width 0) (type default) (color 0 0 0 0))
+  )
   (wire (pts (xy 39.37 160.02) (xy 40.64 160.02))
     (stroke (width 0) (type default) (color 0 0 0 0))
@@
     (stroke (width 0) (type default) (color 0 0 0 0))
   )
-  (wire (pts (xy 212.09 21.59) (xy 212.09 25.4))
+  (wire (pts (xy 212.09 20.32) (xy 212.09 21.59))
     (stroke (width 0) (type default) (color 0 0 0 0))
   )
@@
       (effects (font (size 1.27 1.27)) hide)
     )
+    (pin "1")
+    (pin "2")
+    (pin "3")
     (pin "4")
     (pin "5")
     (pin "6")
+    (pin "10")
+    (pin "8")
+    (pin "9")
+    (pin "11")
+    (pin "12")
+    (pin "13")
+    (pin "14")
+    (pin "7")
   )
   (symbol (lib_id "power:+5V") (at 151.13 21.59 0) (unit 1)
@@
     )
     (property "Datasheet" "" (id 3) (at 229.87 162.56 0)
+      (effects (font (size 1.27 1.27)) hide)
+    )
+    (pin "1")
+  )
+  (symbol (lib_id "power:+BATT") (at 212.09 20.32 0) (unit 1)
+    (in_bom yes) (on_board yes) (fields_autoplaced)
+    (property "Reference" "#PWR011" (id 0) (at 212.09 24.13 0)
+      (effects (font (size 1.27 1.27)) hide)
+    )
+    (property "Value" "+BATT" (id 1) (at 212.09 16.7442 0))
+    (property "Footprint" "" (id 2) (at 212.09 20.32 0)
+      (effects (font (size 1.27 1.27)) hide)
+    )
+    (property "Datasheet" "" (id 3) (at 212.09 20.32 0)
       (effects (font (size 1.27 1.27)) hide)
     )
@@
     (pin "24")
     (pin "25")
+    (pin "26")
     (pin "27")
     (pin "28")
@@
     (pin "2")
     (pin "3")
+    (pin "4")
+    (pin "5")
+    (pin "6")
+    (pin "10")
+    (pin "8")
+    (pin "9")
+    (pin "11")
+    (pin "12")
+    (pin "13")
+    (pin "14")
+    (pin "7")
   )
   (symbol (lib_id "74xx:74LS04") (at 114.3 107.95 0) (unit 5)
@@
       (effects (font (size 1.27 1.27)) hide)
     )
+    (pin "1")
+    (pin "2")
+    (pin "3")
+    (pin "4")
+    (pin "5")
+    (pin "6")
+    (pin "8")
+    (pin "9")
     (pin "10")
     (pin "11")
+    (pin "12")
+    (pin "13")
+    (pin "14")
+    (pin "7")
   )
   (symbol (lib_id "Switch:SW_DIP_x04") (at 104.14 69.85 0) (unit 1)
@@
     (pin "1")
   )
-  (symbol (lib_id "power:+5V") (at 212.09 21.59 0) (unit 1)
-    (in_bom yes) (on_board yes) (fields_autoplaced)
-    (property "Reference" "#PWR011" (id 0) (at 212.09 25.4 0)
-      (effects (font (size 1.27 1.27)) hide)
-    )
-    (property "Value" "+5V" (id 1) (at 212.09 17.9855 0))
-    (property "Footprint" "" (id 2) (at 212.09 21.59 0)
-      (effects (font (size 1.27 1.27)) hide)
-    )
-    (property "Datasheet" "" (id 3) (at 212.09 21.59 0)
-      (effects (font (size 1.27 1.27)) hide)
-    )
-    (pin "1")
-  )
   (symbol (lib_id "Memory_EPROM:27C020") (at 151.13 57.15 0) (unit 1)
     (in_bom yes) (on_board yes) (fields_autoplaced)
@@
       (effects (font (size 1.27 1.27)) hide)
     )
+    (pin "1")
+    (pin "2")
+    (pin "3")
     (pin "4")
     (pin "5")
     (pin "6")
+    (pin "10")
+    (pin "8")
+    (pin "9")
+    (pin "11")
+    (pin "12")
+    (pin "13")
+    (pin "14")
+    (pin "7")
   )
   (symbol (lib_id "gp-parts:Z80-CTC") (at 50.8 139.7 0) (unit 1)
@@
       (effects (font (size 1.27 1.27)) hide)
     )
+    (pin "1")
+    (pin "2")
+    (pin "3")
+    (pin "4")
+    (pin "5")
+    (pin "6")
+    (pin "8")
+    (pin "9")
+    (pin "10")
+    (pin "11")
     (pin "12")
     (pin "13")
+    (pin "14")
+    (pin "7")
   )
   (symbol (lib_id "74xx:74LS00") (at 115.57 163.83 0) (unit 1)
@@
     (pin "2")
     (pin "3")
+    (pin "4")
+    (pin "5")
+    (pin "6")
+    (pin "10")
+    (pin "8")
+    (pin "9")
+    (pin "11")
+    (pin "12")
+    (pin "13")
+    (pin "14")
+    (pin "7")
   )
   (symbol (lib_id "Device:R") (at 168.91 104.14 0) (unit 1)
@@
   )
   (symbol_instances
+    (path "/33d9a8cf-31ed-405a-9422-9faebf8878bc/cf84cf4f-3367-47f1-b6ed-c93da0b3c50b"
+      (reference "#FLG01") (unit 1) (value "PWR_FLAG") (footprint "")
+    )
     (path "/440aa22c-1d00-4ea9-b602-c8241f3dc90e/4223ffb1-b80b-470e-a764-dc8cf9e70297"
       (reference "#FLG0101") (unit 1) (value "PWR_FLAG") (footprint "")
@@
       (reference "#PWR010") (unit 1) (value "GND") (footprint "")
     )
-    (path "/abbd47a0-cbdd-4cdf-93e7-762ec0d28bef"
-      (reference "#PWR011") (unit 1) (value "+5V") (footprint "")
+    (path "/35a78d65-1e29-46bd-8b55-7351f4af17d9"
+      (reference "#PWR011") (unit 1) (value "+BATT") (footprint "")
     )
     (path "/f53a6bc4-f079-44ff-8333-e3b5ae202c06"
@@
       (reference "#PWR071") (unit 1) (value "+5V") (footprint "")
     )
+    (path "/33d9a8cf-31ed-405a-9422-9faebf8878bc/da02eab4-f125-4368-9e3c-c02d2cb40dfa"
+      (reference "#PWR072") (unit 1) (value "+5V") (footprint "")
+    )
+    (path "/33d9a8cf-31ed-405a-9422-9faebf8878bc/b2eb8875-667a-4e5c-af71-f04f8339f5e0"
+      (reference "#PWR073") (unit 1) (value "GND") (footprint "")
+    )
+    (path "/33d9a8cf-31ed-405a-9422-9faebf8878bc/c1e7abff-16d2-4da9-895c-b02ed80bf85e"
+      (reference "#PWR074") (unit 1) (value "+BATT") (footprint "")
+    )
+    (path "/33d9a8cf-31ed-405a-9422-9faebf8878bc/1893df68-fdcb-417f-9ddd-7f6170070c1d"
+      (reference "#PWR075") (unit 1) (value "GND") (footprint "")
+    )
     (path "/440aa22c-1d00-4ea9-b602-c8241f3dc90e/a2c71de6-bb9e-4d92-ba0d-aa77f2d5eb5e"
       (reference "#PWR0101") (unit 1) (value "GND") (footprint "")
@@
       (reference "#PWR0110") (unit 1) (value "GND") (footprint "")
     )
+    (path "/33d9a8cf-31ed-405a-9422-9faebf8878bc/4099d49e-75be-4100-b83d-b3b397a31cac"
+      (reference "BT1") (unit 1) (value "2732 coin cell") (footprint "Battery:BatteryHolder_ComfortableElectronic_CH273-2450_1x2450")
+    )
     (path "/ff65eeb5-1a9d-4f8c-b429-f6027226d0be/5d23be8c-8c8c-4bae-a11d-ee680171dd17"
       (reference "C1") (unit 1) (value "0.01uf") (footprint "Capacitor_THT:C_Disc_D5.0mm_W2.5mm_P5.00mm")
@@
       (reference "D58") (unit 1) (value "LED") (footprint "LED_THT:LED_D3.0mm")
     )
+    (path "/33d9a8cf-31ed-405a-9422-9faebf8878bc/c94ca9b6-b909-473b-9389-1874796b5e96"
+      (reference "D59") (unit 1) (value "1N5817") (footprint "Diode_THT:D_DO-41_SOD81_P10.16mm_Horizontal")
+    )
+    (path "/33d9a8cf-31ed-405a-9422-9faebf8878bc/164e0c90-2306-42a3-9e20-b9ccaf5e6727"
+      (reference "D60") (unit 1) (value "1N4148") (footprint "Diode_THT:D_DO-35_SOD27_P7.62mm_Horizontal")
+    )
     (path "/440aa22c-1d00-4ea9-b602-c8241f3dc90e/cd7599f8-65f2-485b-86c1-3780cd0995d7"
       (reference "J1") (unit 1) (value "Power") (footprint "Connector_PinHeader_2.54mm:PinHeader_1x15_P2.54mm_Vertical")
@@
       (reference "J7") (unit 1) (value "Solenoid") (footprint "Connector_PinHeader_2.54mm:PinHeader_1x09_P2.54mm_Vertical")
     )
+    (path "/33d9a8cf-31ed-405a-9422-9faebf8878bc/d6d585b8-399f-4079-b82d-ec7e073560f0"
+      (reference "J8") (unit 1) (value "Ext Battery") (footprint "Connector_PinHeader_2.54mm:PinHeader_1x03_P2.54mm_Vertical")
+    )
     (path "/440aa22c-1d00-4ea9-b602-c8241f3dc90e/f094855b-7c38-41a8-88b2-dec9e55db250"

Commit message: Update BDU connector
Changed lines of the file:
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@@
   (title_block
     (title "CPU and Memory")
-    (date "2022-02-05")
-    (rev "1.1")
+    (date "2022-08-27")
+    (rev "1.5")
     (company "ePinball")
     (comment 1 "github.com/jfleitz/gp-mpu")
@@
   (symbol (lib_id "Memory_NVRAM:FM16W08-SG") (at 212.09 45.72 0) (unit 1)
     (in_bom yes) (on_board yes) (fields_autoplaced)
-    (property "Reference" "U7" (id 0) (at 214.1094 25.2435 0)
+    (property "Reference" "U7" (id 0) (at 214.1094 64.2604 0)
       (effects (font (size 1.27 1.27)) (justify left))
     )
-    (property "Value" "FM16W08-SG" (id 1) (at 214.1094 28.0186 0)
+    (property "Value" "FM16W08-SG" (id 1) (at 214.1094 66.7973 0)
       (effects (font (size 1.27 1.27)) (justify left))
     )
@@
     )
   )
-  (sheet (at 435.61 99.06) (size 41.91 34.29) (fields_autoplaced)
+  (sheet (at 439.42 95.25) (size 34.29 41.91) (fields_autoplaced)
     (stroke (width 0.1524) (type solid) (color 0 0 0 0))
     (fill (color 0 0 0 0.0000))
-    (property "Sheet name" "ports" (id 0) (at 435.61 98.3484 0)
+    (property "Sheet name" "ports" (id 0) (at 439.42 94.5384 0)
       (effects (font (size 1.27 1.27)) (justify left bottom))
     )
-    (property "Sheet file" "ports.kicad_sch" (id 1) (at 435.61 133.9346 0)
+    (property "Sheet file" "ports.kicad_sch" (id 1) (at 439.42 137.7446 0)
       (effects (font (size 1.27 1.27)) (justify left top))
     )
@@
       (reference "J9") (unit 1) (value "DISPLAY") (footprint "gp-connector:display-upright")
     )
+    (path "/33d9a8cf-31ed-405a-9422-9faebf8878bc/d22ae9a6-0fb5-4f30-9348-0c22d164c7ee"
+      (reference "JP1") (unit 1) (value "NVRAM") (footprint "Jumper:SolderJumper-2_P1.3mm_Open_RoundedPad1.0x1.5mm")
+    )
     (path "/a452fa18-3a10-4a3a-b908-f3e47e22c275/b1537c9a-ac6c-4856-a0b0-594671ca4ebd"
