File: powerpins.kicad_sch (KiCad schematic)
At the start: 15 parts, among them U12 74LS00, U16 LM339, U19 LM339, U20 LM339, U3 74LS04, U4 74LS32, U5 74LS00

Commit message: updates
Parts:
- added BT1: (no value), Battery:BatteryHolder_ComfortableElectronic_CH273-2450_1x2450, symbol Device:Battery_Cell
- added D59: 1N5817, Diode_THT:D_DO-41_SOD81_P10.16mm_Horizontal, symbol Diode:1N5817
- added D60: 1N4148, Diode_THT:D_DO-35_SOD27_P7.62mm_Horizontal, symbol Diode:1N4148
- added J8: Ext Battery, Connector_PinHeader_2.54mm:PinHeader_1x03_P2.54mm_Vertical, symbol Connector:Conn_01x03_Male
Connections:
- net +5V: now also D59.2 (A)
- net GND: now also BT1.2 (-), J8.1 (Pin_1), J8.3 (Pin_3)
- new net: BT1.1 (+), D60.2 (A), J8.2 (Pin_2)
- new net +BATT: D59.1 (K), D60.1 (K)
- no-connect marks 2 -> 7
Other:
- note added: "Battery backup when using a 6264 vs NVRAM. If using NVRAM, install a jumper at D59, and don't install the other components"

Commit message: Update BDU connector
Parts:
- added JP1: NVRAM, Jumper:SolderJumper-2_P1.3mm_Open_RoundedPad1.0x1.5mm, symbol Jumper:SolderJumper_2_Open
- BT1: value (none) -> 2732 coin cell
Connections:
- net +5V: now also JP1.2 (B)
- net +BATT: now also JP1.1 (A)
Changed lines of the file:
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@@
   (title_block
     (title "Power and Non-Connected pins")
-    (date "2022-02-05")
-    (rev "1.1")
+    (date "2022-08-27")
+    (rev "1.5")
     (company "ePinball")
     (comment 1 "github.com/jfleitz/gp-mpu")
@@
   )
   (junction (at 35.56 135.89) (diameter 0) (color 0 0 0 0)
+  )
+  (junction (at 121.92 31.75) (diameter 0) (color 0 0 0 0)
   )
   (junction (at 233.68 128.27) (diameter 0) (color 0 0 0 0)
@@
     (stroke (width 0) (type default) (color 0 0 0 0))
   )
-  (wire (pts (xy 121.92 29.21) (xy 121.92 33.02))
+  (wire (pts (xy 121.92 29.21) (xy 121.92 31.75))
     (stroke (width 0) (type default) (color 0 0 0 0))
   )
@@
     (stroke (width 0) (type default) (color 0 0 0 0))
   )
+  (wire (pts (xy 110.49 43.18) (xy 110.49 40.64))
+    (stroke (width 0) (type default) (color 0 0 0 0))
+  )
   (wire (pts (xy 233.68 123.19) (xy 233.68 128.27))
     (stroke (width 0) (type default) (color 0 0 0 0))
@@
     (stroke (width 0) (type default) (color 0 0 0 0))
   )
+  (wire (pts (xy 110.49 33.02) (xy 110.49 31.75))
+    (stroke (width 0) (type default) (color 0 0 0 0))
+  )
   (wire (pts (xy 233.68 67.31) (xy 233.68 74.93))
     (stroke (width 0) (type default) (color 0 0 0 0))
@@
     (stroke (width 0) (type default) (color 0 0 0 0))
   )
+  (wire (pts (xy 121.92 31.75) (xy 121.92 33.02))
+    (stroke (width 0) (type default) (color 0 0 0 0))
+  )
   (wire (pts (xy 121.92 40.64) (xy 121.92 43.18))
     (stroke (width 0) (type default) (color 0 0 0 0))
@@
     (stroke (width 0) (type default) (color 0 0 0 0))
   )
+  (wire (pts (xy 110.49 43.18) (xy 121.92 43.18))
+    (stroke (width 0) (type default) (color 0 0 0 0))
+  )
   (wire (pts (xy 233.68 118.11) (xy 233.68 123.19))
     (stroke (width 0) (type default) (color 0 0 0 0))
@@
   )
   (wire (pts (xy 121.92 62.23) (xy 121.92 64.77))
+    (stroke (width 0) (type default) (color 0 0 0 0))
+  )
+  (wire (pts (xy 110.49 31.75) (xy 121.92 31.75))
     (stroke (width 0) (type default) (color 0 0 0 0))
   )
@@
       (effects (font (size 1.27 1.27)) (justify left))
     )
-    (property "Value" "" (id 1) (at 124.841 59.3602 0)
+    (property "Value" "2732 coin cell" (id 1) (at 124.841 59.3602 0)
       (effects (font (size 1.27 1.27)) (justify left))
     )
@@
     (pin "1")
   )
+  (symbol (lib_id "Jumper:SolderJumper_2_Open") (at 110.49 36.83 90) (unit 1)
+    (in_bom yes) (on_board yes) (fields_autoplaced)
+    (property "Reference" "JP1" (id 0) (at 112.141 35.9953 90)
+      (effects (font (size 1.27 1.27)) (justify right))
+    )
+    (property "Value" "NVRAM" (id 1) (at 112.141 38.5322 90)
+      (effects (font (size 1.27 1.27)) (justify right))
+    )
+    (property "Footprint" "Jumper:SolderJumper-2_P1.3mm_Open_RoundedPad1.0x1.5mm" (id 2) (at 110.49 36.83 0)
+      (effects (font (size 1.27 1.27)) hide)
+    )
+    (property "Datasheet" "~" (id 3) (at 110.49 36.83 0)
+      (effects (font (size 1.27 1.27)) hide)
+    )
+    (pin "1")
+    (pin "2")
+  )
   (symbol (lib_id "Connector:Conn_01x03_Male") (at 153.67 54.61 180) (unit 1)
